File: Hardware/mainboarddesign/mainboarddesign.kicad_sch (KiCad schematic)
At the start: 3 parts, among them U1 ESP32-S3-DEVKITC-1U-N8R2

Commit message: Added more stuff for the ESP and UWB
Parts:
- added U4: ~, symbol ESP32-Symbols:X9313
Connections:
- net +3V3: now also U4. (Vss)
- net GND: now also U4. (Vss)
- net at U2. (KEY/IGN): now also U4. (Vss)
- net X9313_CS: now reaches U1.J1_4 (GPIO4)
- net X9313_CS: now also U4. (Vss)
- net X9313_INC: now reaches U1.J1_5 (GPIO5)
- net X9313_INC: now also U4. (Vss)
- net X9313_U/D: now reaches U1.J1_6 (GPIO6)
- net X9313_U/D: now also U4. (Vss)
- new net: U2. (KEY/IGN), U4. (Vss) (x2)
