File: Hardware/Main_Board/Connectors.kicad_sch (KiCad schematic)
At the start: 0 parts

Commit message: Added all the main connectors
Parts:
- added J1, J2: Conn_01x22_Socket, Connector_PinSocket_2.54mm:PinSocket_1x22_P2.54mm_Vertical, symbol Connector:Conn_01x22_Socket
- added J3: Conn_01x07_Socket, symbol Connector:Conn_01x07_Socket
- added J4: Conn_01x04_Socket, symbol Connector:Conn_01x04_Socket
- added J5: Conn_01x03_Socket, symbol Connector:Conn_01x03_Socket
- added U1: ~, symbol ESP32-Symbols:Battery_Connector
- added U4, U6: ~, symbol ESP32-Symbols:X9313
- added U5, U7: ~, symbol ESP32-Symbols:MotoController
Connections:
- new net: U4. (Vss), U5. (KEY/IGN) (x3)
- new net: U6. (Vss), U7. (KEY/IGN) (x3)
- new net +3V3: U4. (Vss), U6. (Vss)
- new net 36v: U1. (Pin2)
- new net 3V3: J2.1 (Pin_1), J2.2 (Pin_2), J5.2 (Pin_2)
- new net 5VO: J2.21 (Pin_21), J3.1 (Pin_1), J3.2 (Pin_2), J4.1 (Pin_1)
- new net GND: J1.1 (Pin_1), J1.21 (Pin_21), J1.22 (Pin_22), J2.22 (Pin_22), J3.3 (Pin_3), J4.4 (Pin_4), J5.1 (Pin_1), U1. (Pin2), U4. (Vss), U6. (Vss)
- new net GPIO0: J1.14 (Pin_14)
- new net GPIO1: J1.4 (Pin_4)
- new net GPIO10: J2.16 (Pin_16)
- new net GPIO11: J2.17 (Pin_17)
- new net GPIO12: J2.18 (Pin_18)
- new net GPIO13: J2.19 (Pin_19)
- new net GPIO14: J2.20 (Pin_20), J5.3 (Pin_3)
- new net GPIO15: J2.8 (Pin_8), J4.2 (Pin_2)
- new net GPIO16: J2.9 (Pin_9), J4.3 (Pin_3)
- new net GPIO17: J2.10 (Pin_10), J3.6 (Pin_6)
- new net GPIO18: J2.11 (Pin_11), J3.7 (Pin_7)
- new net GPIO19: J1.20 (Pin_20)
- new net GPIO2: J1.5 (Pin_5)
- new net GPIO20: J1.19 (Pin_19)
- new net GPIO21: J1.18 (Pin_18)
- new net GPIO3: J2.13 (Pin_13)
- new net GPIO35: J1.13 (Pin_13)
- new net GPIO36: J1.12 (Pin_12)
- new net GPIO37: J1.11 (Pin_11)
- new net GPIO38: J1.10 (Pin_10)
- new net GPIO39: J1.9 (Pin_9)
- new net GPIO4: J2.4 (Pin_4)
- new net GPIO40: J1.8 (Pin_8)
- new net GPIO41: J1.7 (Pin_7)
- new net GPIO42: J1.6 (Pin_6)
- new net GPIO43: J1.2 (Pin_2), J3.4 (Pin_4)
- new net GPIO44: J1.3 (Pin_3), J3.5 (Pin_5)
- new net GPIO45: J1.15 (Pin_15)
- new net GPIO46: J2.14 (Pin_14)
- new net GPIO47: J1.17 (Pin_17)
- new net GPIO48: J1.16 (Pin_16)
- new net GPIO5: J2.5 (Pin_5)
- new net GPIO6: J2.6 (Pin_6)
- new net GPIO7: J2.7 (Pin_7)
- new net GPIO8: J2.12 (Pin_12)
- new net GPIO9: J2.15 (Pin_15)
- new net RST: J2.3 (Pin_3)
- new net X9313_CS: U4. (Vss), U6. (Vss)
- new net X9313_INC: U4. (Vss), U6. (Vss)
- new net X9313_U/D: U4. (Vss), U6. (Vss)
Other:
- note added: "Battery Connector"
- note added: "ESP CONNECTOR"
- note added: "Extra parts to be determined"
- note added: "LIDAR CONNECTOR"
- note added: "MOTOR CONTROLLER CONECTOR"
- note added: "RF MODULE CONNECTOR"
