File: Hardware/Main_Board/Connectors.kicad_sch (KiCad schematic)
At the start: 0 parts

Commit message: added gerbers, drill files, BOM and CPL for the main board
Parts:
- added J2, J3: Conn_01x22_Socket, Connector_PinSocket_2.54mm:PinSocket_1x22_P2.54mm_Vertical, symbol Connector:Conn_01x22_Socket
- added J4, J5: Conn_01x08_Socket, Connector_PinSocket_2.54mm:PinSocket_1x08_P2.54mm_Vertical, symbol Connector:Conn_01x08_Socket
- added J6: Conn_01x05_Socket, Connector_PinSocket_2.54mm:PinSocket_1x05_P2.54mm_Vertical, symbol Connector:Conn_01x05_Socket
Connections:
- new net 5V0: J2.2 (Pin_2)
- new net CLK: J4.2 (Pin_2)
- new net CS: J4.5 (Pin_5)
- new net EXTON: J5.1 (Pin_1)
- new net GND: J2.1 (Pin_1), J3.1 (Pin_1), J3.2 (Pin_2), J3.22 (Pin_22), J6.2 (Pin_2)
- new net GPIO0: J3.9 (Pin_9)
- new net GPIO1: J3.19 (Pin_19)
- new net GPIO10: J2.7 (Pin_7)
- new net GPIO11: J2.6 (Pin_6)
- new net GPIO12: J2.5 (Pin_5)
- new net GPIO13: J2.4 (Pin_4)
- new net GPIO14: J2.3 (Pin_3)
- new net GPIO15: J2.15 (Pin_15)
- new net GPIO16: J2.14 (Pin_14)
- new net GPIO17: J2.13 (Pin_13)
- new net GPIO18: J2.12 (Pin_12)
- new net GPIO19: J3.3 (Pin_3)
- new net GPIO2: J3.18 (Pin_18)
- new net GPIO20: J3.4 (Pin_4)
- new net GPIO21: J3.5 (Pin_5)
- new net GPIO3: J2.10 (Pin_10)
- new net GPIO35: J3.10 (Pin_10)
- new net GPIO36: J3.11 (Pin_11)
- new net GPIO37: J3.12 (Pin_12)
- new net GPIO38: J3.13 (Pin_13)
- new net GPIO39: J3.14 (Pin_14)
- new net GPIO4: J2.19 (Pin_19)
- new net GPIO40: J3.15 (Pin_15)
- new net GPIO41: J3.16 (Pin_16)
- new net GPIO42: J3.17 (Pin_17)
- new net GPIO43: J3.21 (Pin_21)
- new net GPIO44: J3.20 (Pin_20)
- new net GPIO45: J3.8 (Pin_8)
- new net GPIO46: J2.9 (Pin_9)
- new net GPIO47: J3.6 (Pin_6)
- new net GPIO48: J3.7 (Pin_7)
- new net GPIO5: J2.18 (Pin_18)
- new net GPIO6: J2.17 (Pin_17)
- new net GPIO7: J2.16 (Pin_16)
- new net GPIO8: J2.11 (Pin_11)
- new net GPIO9: J2.8 (Pin_8)
- new net IRQ: J4.1 (Pin_1)
- new net MISO: J4.3 (Pin_3)
- new net MOSI: J4.4 (Pin_4)
- new net RF_RX: J6.3 (Pin_3)
- new net RF_TX: J6.4 (Pin_4)
- new net RST: J2.20 (Pin_20)
- new net SET: J6.5 (Pin_5)
- new net VDD3V3: J6.1 (Pin_1)
- new net WAKEUP: J5.2 (Pin_2)
- new net uGPIO0: J4.6 (Pin_6)
- new net uGPIO1: J4.7 (Pin_7)
- new net uGPIO2: J4.8 (Pin_8)
- new net uGPIO3: J5.8 (Pin_8)
- new net uGPIO4: J5.7 (Pin_7)
- new net uGPIO5: J5.6 (Pin_6)
- new net uGPIO6: J5.5 (Pin_5)
- new net uGPIO7: J5.4 (Pin_4)
- new net ~{RST}: J5.3 (Pin_3)
- no-connect marks 0 -> 2
Other:
- note added: "ESP32 Connectors"
- note added: "Global/Hierarchical Labels"
- note added: "RF Transceiver Connector"
- note added: "UWB Connectors"
