File: Hardware/Main_Board/ESP32S3.kicad_sch (KiCad schematic)
At the start: 4 parts, among them U1 ESP32-S3-DEVKITC-1U-N8R2

Commit message: Added all the main connectors
Parts:
- removed U4: ~, symbol ESP32-Symbols:X9313
- removed U5: ~, symbol ESP32-Symbols:MotoController
Other:
- note removed: "Extra parts to be determined"
