File: Hardware/Main_Board/DWM1000.kicad_sch (KiCad schematic)
At the start: 0 parts

Commit message: finished most of the main board
Parts:
- added U4: ~, ESP32-footprints:STM32N6_Board, symbol ESP32-Symbols:STM32N6_Board
Connections:
- new net 5V: U4.1 (5V), U4.17 (5V), U4.20 (5V), U4.36 (5V)
- new net CLK1: U4.10 (CLK1)
- new net CLK5: U4.27 (CLK5)
- new net GND: U4.18 (GND), U4.19 (GND), U4.2 (GND), U4.35 (GND), U4.GND1 (GND), U4.GND2 (GND), U4.GND3 (GND), U4.GND4 (GND)
- new net MISO1: U4.7 (MISO1)
- new net MISO5: U4.30 (MISO5)
- new net MOSI1: U4.8 (MOSI1)
- new net MOSI5: U4.29 (MOSI5)
- new net PA10: U4.13 (PA10)
- new net PA15: U4.14 (PA15)
- new net PC7: U4.15 (PC7)
- new net PD13: U4.21 (PD13)
- new net PF14: U4.23 (PF14)
- new net PF7: U4.22 (PF7)
- new net PG13: U4.16 (PG13)
- new net PG15: U4.24 (PG15)
- new net RX1: U4.4 (RX1)
- new net RX2: U4.33 (RX2)
- new net RX3: U4.6 (RX3)
- new net RX4: U4.31 (RX4)
- new net SCL1: U4.12 (SCL1)
- new net SCL2: U4.25 (SCL2)
- new net SDA1: U4.11 (SDA1)
- new net SDA2: U4.26 (SDA2)
- new net TX1: U4.3 (TX1)
- new net TX2: U4.34 (TX2)
- new net TX3: U4.5 (TX3)
- new net TX4: U4.32 (TX4)
- new net ~{CS}1: U4.9 (~{CS}1)
- new net ~{CS}5: U4.28 (~{CS}5)

Commit message: added gerbers, drill files, BOM and CPL for the main board
Parts:
- removed U4: ~, ESP32-footprints:STM32N6_Board, symbol ESP32-Symbols:STM32N6_Board
