File: Hardware/Main_Board/Main_Board.kicad_pcb (KiCad board)
At the start: 2 copper layers, 15 parts, among them J1 Conn_01x02_Socket, U1 ESP32-S3-DEVKITC-1U-N8R2, U2 LM2596DSADJG, U3 DWM1000

Commit message: added gerbers, drill files, BOM and CPL for the main board
Parts:
- removed C3: C, Capacitor_SMD:C_0805_2012Metric
- added G***: LOGO, ESP32-footprints:SolarVisionMowerLogo, F.Cu at (115.9, 115.5)
- added J2: Conn_01x22_Socket, Connector_PinSocket_2.54mm:PinSocket_1x22_P2.54mm_Vertical, F.Cu at (97.3, 66.8)
- added J3: Conn_01x22_Socket, Connector_PinSocket_2.54mm:PinSocket_1x22_P2.54mm_Vertical, F.Cu at (63.2, 66.9)
- added J4: Conn_01x08_Socket, Connector_PinSocket_2.54mm:PinSocket_1x08_P2.54mm_Vertical, F.Cu at (141.7, 58.0)
- added J5: Conn_01x08_Socket, Connector_PinSocket_2.54mm:PinSocket_1x08_P2.54mm_Vertical, F.Cu at (111.7, 58.0)
- added J6: Conn_01x05_Socket, Connector_PinSocket_2.54mm:PinSocket_1x05_P2.54mm_Vertical, F.Cu at (73.6, 135.0)
- added REF**: MountingHole_2.5mm_Pad, MountingHole:MountingHole_2.5mm_Pad, F.Cu at (249.8, 135.2)
- added REF**: MountingHole_2.5mm_Pad, MountingHole:MountingHole_2.5mm_Pad, F.Cu at (57.5, 54.4)
- added REF**: MountingHole_2.5mm_Pad, MountingHole:MountingHole_2.5mm_Pad, F.Cu at (249.8, 54.4)
- added REF**: MountingHole_2.5mm_Pad, MountingHole:MountingHole_2.5mm_Pad, F.Cu at (57.5, 135.2)
- D1: moved to B.Cu
- L1: footprint Inductor_SMD:L_0603_1608Metric -> Inductor_SMD:L_0805_2012Metric
- moved J1 177.6 mm to (98.5, 135.2)
- moved C1 174.9 mm to (116.1, 127.1), turned to -90 degrees
- moved C2 164.1 mm to (129.9, 83.2), turned to 90 degrees
- moved U5 163.1 mm to (137.9, 83.2), turned to 180 degrees
- moved D1 160.7 mm to (126.1, 129.8), turned to -90 degrees
- moved R2 148.7 mm to (122.2, 129.9), turned to 90 degrees
- moved R1 148.7 mm to (122.2, 126.4), turned to 90 degrees
- moved R4 145.8 mm to (133.2, 81.2), turned to -90 degrees
- moved L1 144.9 mm to (126.1, 125.5), turned to 180 degrees
- moved R3 143.8 mm to (133.2, 85.0), turned to -90 degrees
- moved U1 29.1 mm to (80.1, 90.3), turned to 180 degrees
- moved U2 25.9 mm to (137.4, 127.3)
- moved U4 14.4 mm to (201.2, 96.2)
- moved U3 9.09 mm to (126.7, 53.5)
Connections:
- net /ESP32S3/GPIO10 renamed /Connectors/GPIO10
- net /ESP32S3/GPIO11 renamed /Connectors/GPIO11
- net /ESP32S3/GPIO12 renamed /Connectors/GPIO12
- net /ESP32S3/GPIO13 renamed /Connectors/GPIO13
- net /STM32N6/CLK1 renamed /Connectors/CLK1
- net /STM32N6/CLK5 renamed /Connectors/CLK5
- net /STM32N6/MISO1 renamed /Connectors/MISO1
- net /STM32N6/MISO5 renamed /Connectors/MISO5
- net /STM32N6/MOSI1 renamed /Connectors/MOSI1
- net /STM32N6/MOSI5 renamed /Connectors/MOSI5
- net /STM32N6/PA10 renamed /Connectors/PA10
- net /STM32N6/PA15 renamed /Connectors/PA15
- net /STM32N6/PC7 renamed /Connectors/PC7
- net /STM32N6/PD13 renamed /Connectors/PD13
- net /STM32N6/PF14 renamed /Connectors/PF14
- net /STM32N6/PF7 renamed /Connectors/PF7
- net /STM32N6/PG13 renamed /Connectors/PG13
- net /STM32N6/PG15 renamed /Connectors/PG15
- net /STM32N6/RX2 renamed /Connectors/RX2
- net /STM32N6/RX3 renamed /Connectors/RX3
- net /STM32N6/RX4 renamed /Connectors/RX4
- net /STM32N6/SCL1 renamed /Connectors/SCL1
- net /STM32N6/SCL2 renamed /Connectors/SCL2
- net /STM32N6/SDA1 renamed /Connectors/SDA1
- net /STM32N6/SDA2 renamed /Connectors/SDA2
- net /STM32N6/TX2 renamed /Connectors/TX2
- net /STM32N6/TX3 renamed /Connectors/TX3
- net /STM32N6/TX4 renamed /Connectors/TX4
- net /STM32N6/~{CS}1 renamed /Connectors/~{CS}1
- net /STM32N6/~{CS}5 renamed /Connectors/~{CS}5
- U1 pad J1_10: /ESP32S3/GPIO17 -> /Connectors/GPIO17
- U1 pad J1_11: /ESP32S3/GPIO18 -> /Connectors/GPIO18
- U1 pad J1_12: /ESP32S3/GPIO8 -> /Connectors/GPIO8
- U1 pad J1_13: /ESP32S3/GPIO3 -> /Connectors/GPIO3
- U1 pad J1_14: /ESP32S3/GPIO46 -> /Connectors/GPIO46
- U1 pad J1_15: /ESP32S3/GPIO9 -> /Connectors/GPIO9
- U1 pad J1_20: /ESP32S3/GPIO14 -> /Connectors/GPIO14
- U1 pad J1_3: /ESP32S3/RST -> /Connectors/RST
- U1 pad J1_4: /ESP32S3/GPIO4 -> /Connectors/GPIO4
- U1 pad J1_5: /ESP32S3/GPIO5 -> /Connectors/GPIO5
- U1 pad J1_6: /ESP32S3/GPIO6 -> /Connectors/GPIO6
- U1 pad J1_7: /ESP32S3/GPIO7 -> /Connectors/GPIO7
- U1 pad J1_8: /ESP32S3/GPIO15 -> /Connectors/GPIO15
- U1 pad J1_9: /ESP32S3/GPIO16 -> /Connectors/GPIO16
- U1 pad J3_10: /ESP32S3/GPIO38 -> /Connectors/GPIO38
- U1 pad J3_11: /ESP32S3/GPIO37 -> /Connectors/GPIO37
- U1 pad J3_12: /ESP32S3/GPIO36 -> /Connectors/GPIO36
- U1 pad J3_13: /ESP32S3/GPIO35 -> /Connectors/GPIO35
- U1 pad J3_14: /ESP32S3/GPIO0 -> /Connectors/GPIO0
- U1 pad J3_15: /ESP32S3/GPIO45 -> /Connectors/GPIO45
- U1 pad J3_16: /ESP32S3/TX1 -> /Connectors/TX1
- U1 pad J3_17: /ESP32S3/RX1 -> /Connectors/RX1
- U1 pad J3_18: /ESP32S3/GPIO21 -> /Connectors/GPIO21
- U1 pad J3_19: /ESP32S3/GPIO20 -> /Connectors/GPIO20
- U1 pad J3_2: /ESP32S3/GPIO43 -> /Connectors/GPIO43
- U1 pad J3_20: /ESP32S3/GPIO19 -> /Connectors/GPIO19
- U1 pad J3_3: /ESP32S3/GPIO44 -> /Connectors/GPIO44
- U1 pad J3_4: /ESP32S3/GPIO1 -> /Connectors/GPIO1
- U1 pad J3_5: /ESP32S3/GPIO2 -> /Connectors/GPIO2
- U1 pad J3_6: /ESP32S3/GPIO42 -> /Connectors/GPIO42
- U1 pad J3_7: /ESP32S3/GPIO41 -> /Connectors/GPIO41
- U1 pad J3_8: /ESP32S3/GPIO40 -> /Connectors/GPIO40
- U1 pad J3_9: /ESP32S3/GPIO39 -> /Connectors/GPIO39
- U3 pad 1: /ESP32S3/EXTON -> /Connectors/EXTON
- U3 pad 10: /ESP32S3/GPIO5 -> /Connectors/uGPIO5
- U3 pad 11: /ESP32S3/GPIO4 -> /Connectors/uGPIO4
- U3 pad 12: /ESP32S3/GPIO3 -> /Connectors/uGPIO3
- U3 pad 13: /ESP32S3/GPIO2 -> /Connectors/uGPIO2
- U3 pad 14: /ESP32S3/GPIO1 -> /Connectors/uGPIO1
- U3 pad 15: /ESP32S3/GPIO0 -> /Connectors/uGPIO0
- U3 pad 2: /ESP32S3/WAKEUP -> /Connectors/WAKEUP
- U3 pad 22: /ESP32S3/IRQ -> /Connectors/IRQ
- U3 pad 3: /ESP32S3/~{RST} -> /Connectors/~{RST}
- U3 pad 4: /ESP32S3/GPIO7 -> /Connectors/uGPIO7
- U3 pad 9: /ESP32S3/GPIO6 -> /Connectors/uGPIO6
- U4 pad 3: /STM32N6/TX1 -> /Connectors/TX1
- U4 pad 4: /STM32N6/RX1 -> /Connectors/RX1
Routing:
- net VDD3V3: track 0.00 -> 175.0 mm, vias 0 -> 6
- net /Connectors/RX1: track 0.00 -> 122.4 mm
- net /Connectors/TX1: track 0.00 -> 114.9 mm
- net /Connectors/GPIO12: track 0.00 -> 77.2 mm
- net /Connectors/GPIO10: track 0.00 -> 77.2 mm
- net /Connectors/GPIO11: track 0.00 -> 75.4 mm
- net /Connectors/GPIO13: track 0.00 -> 70.2 mm
- net /Connectors/GPIO7: track 0.00 -> 41.1 mm
- net /Connectors/GPIO6: track 0.00 -> 37.5 mm
- net GND: track 0.00 -> 34.9 mm, vias 0 -> 1
- net +BATT: track 0.00 -> 34.3 mm
- net /Connectors/GPIO5: track 0.00 -> 33.9 mm
- net /Connectors/uGPIO2: track 0.00 -> 19.5 mm
- net /Connectors/uGPIO3: track 0.00 -> 19.5 mm
- net /Connectors/uGPIO1: track 0.00 -> 17.0 mm
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- added copper zone on B.Cu, net 5V0
- added copper zone on F.Cu, net GND
- added copper zone on F.Cu, net Net-(U2-FEEDBACK)
- added copper zone on F.Cu, net Net-(U5-ADJ)
- added copper zone on B.Cu, net VDD3V3
Other:
- board outline added: 200.3 x 88.8 mm
- board text added: "Main Logic Board for the SolarVision Mower Rev A - 03/2026 SolarVisionMower.github.io"
