File: Hardware/STM32N6_Board/Connectors.kicad_sch (KiCad schematic)
At the start: 17 parts, among them J10 BOOT0, J11 Conn_01x18_Socket, J12 Conn_01x18_Socket, J3 Conn_01x08_Pin, J4 Conn_01x18_Pin, J5 Conn_01x18_Pin, J6 Conn_01x05_Pin, J7 SFW15R-2STE1LF, J8 12401832E402A, J9 BOOT1

Commit message: almost finished with the board
Parts:
- removed J8: 12401832E402A, STM32N6_Footprints:AMPHENOL_12401832E402A, symbol STM32N6_Symbols:12401832E402A
- added J13: TYPE-C_16PIN_2MD__073_, STM32N6_Footprints:SHOUHAN_TYPE-C_16PIN_2MD__073_, symbol STM32N6_Symbols:TYPE-C_16PIN_2MD__073_
Connections:
- net CC1: now also J13.A5 (CC1)
- net CC2: now also J13.B5 (CC2)
- net GND: now also J13.A1_B12 (GND_A), J13.B1_A12 (GND_B), J13.SH1 (SHIELD), J13.SH2 (SHIELD), J13.SH3 (SHIELD), J13.SH4 (SHIELD)
- net I2C1_SCL: no longer J7.13
- net I2C1_SDA: no longer J7.14
- net I2C2_SCL: now also J7.13
- net I2C2_SDA: now also J7.14
- net TIM1_CH4: now also J11.13 (Pin_13), J4.13 (Pin_13); no longer J12.14 (Pin_14), J5.14 (Pin_14)
- net TIM2_CH1: now also J12.14 (Pin_14), J5.14 (Pin_14); no longer J11.13 (Pin_13), J4.13 (Pin_13)
- net TIM3_CH3: now also J11.15 (Pin_15), J4.15 (Pin_15); no longer J12.16 (Pin_16), J5.16 (Pin_16)
- net TIM4_CH1: now also J12.16 (Pin_16), J5.16 (Pin_16); no longer J11.15 (Pin_15), J4.15 (Pin_15)
- new net HSD_N: J13.A7 (DN1), J13.B7 (DN2)
- new net HSD_P: J13.A6 (DP1), J13.B6 (DP2)
- new net VBUS: J13.A4_B9 (VBUS_A), J13.B4_A9 (VBUS_B)
- no-connect marks 10 -> 3
