File: Hardware/STM32N6_Board/Power_Unit.kicad_sch (KiCad schematic)
At the start: 72 parts, among them J1 Conn_01x02_Pin, J2 Conn_01x02_Pin, U1 STM32N657I0H3Q, U2 SPX5205-ADJ, U3 SPX5205-ADJ, U4 SPX5205-ADJ, U5 SPX5205-ADJ, U6 MC34064-ADJ-TR

Commit message: almost finished with the board
Parts:
- removed C2: 2.2n, Capacitor_SMD:C_0402_1005Metric, symbol Device:C_Small_US
- removed C6: 15u, Capacitor_SMD:C_0402_1005Metric, symbol Device:C_Small_US
- removed J2: Conn_01x02_Pin, Connector_PinHeader_2.54mm:PinHeader_1x02_P2.54mm_Vertical, symbol Connector:Conn_01x02_Pin
- removed L1: 1u, Inductor_SMD:L_1206_3216Metric_Pad1.42x1.75mm_HandSolder, symbol Device:L_Small
- removed R2: 2, Resistor_SMD:R_0402_1005Metric, symbol Device:R_Small_US
- added D10, D8, D9: D_TVS, LED_SMD:LED_0805_2012Metric_Pad1.15x1.40mm_HandSolder, symbol Device:D_TVS
- added FB2: 70R@100M, Inductor_SMD:L_1206_3216Metric_Pad1.42x1.75mm_HandSolder, symbol Device:FerriteBead_Small
Connections:
- net VFBSMPS is gone; now on net VDDCORE: C3.1, C35.1, C4.1, C5.1, U1.D2 (VFBSMPS)
- net +5V: now also D7.2 (A2), D10.2 (A2), D8.2 (A2), D9.2 (A2); no longer D7.1 (A1)
- net GND: now also D7.1 (A1), D10.1 (A1), D8.1 (A1), D9.1 (A1); no longer D7.2 (A2)
- net VDDCORE: now also FB2.2
- net VLXSMPS: now also FB2.1
Other:
- moved on the sheet: D7
