File: Hardware/STM32N6_Board/STM32N6_Board.kicad_pcb (KiCad board)
At the start: 6 copper layers, 82 x 78.7 mm, 151 parts, among them J1 Conn_01x02_Pin, J10 BOOT0, J11 Conn_01x18_Socket, J12 Conn_01x18_Socket, J13 TYPE-C_16PIN_2MD__073_, J3 Conn_01x08_Pin, J4 Conn_01x18_Pin, J5 Conn_01x18_Pin, J6 Conn_01x05_Pin, J7 SFW15R-2STE1LF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

Commit message: Added the gerbers, drill files, BOM, and CPL files
Parts:
- removed D12: D_TVS, LED_SMD:LED_0805_2012Metric_Pad1.15x1.40mm_HandSolder
- added D11: D_TVS_Dual_AAC, Package_TO_SOT_SMD:SOT-723, F.Cu at (175.8, 109.2)
- C38: value 470u -> 100u
- D10, D4, D7, D8, D9: value D_TVS -> D_TVS_Dual_AAC; footprint LED_SMD:LED_0805_2012Metric_Pad1.15x1.40mm_HandSolder -> Package_TO_SOT_SMD:SOT-723
- moved D7 1.13 mm to (157.5, 96.0), turned to 90 degrees
- moved D9 0.81 mm to (222.5, 96.0), turned to 90 degrees
- moved D8 0.30 mm to (157.5, 146.7), turned to -90 degrees
- moved D10 0.25 mm to (222.5, 146.7), turned to -90 degrees
- moved D4 0.16 mm to (198.7, 150.7), turned to -90 degrees
Connections:
- D10 pad 1: GND -> +5V
- D4 pad 1: GND -> /Analog_Unit/VBUS
- D7 pad 1: GND -> +5V
- D8 pad 1: GND -> +5V
- D9 pad 1: GND -> +5V
Routing:
- net GND: track 102.6 -> 104.8 mm, vias 68 -> 69
- net /XSPI NOR Flash/VDD_OCTO: track 28.2 -> 29.5 mm
- net +5V: track 23.5 -> 22.8 mm, vias 20 -> 16
Other:
- board text added: "1v8_AON"
- board text added: "5V"
- board text added: "CLK1"
- board text added: "CLK5"
- board text added: "GND"
- board text added: "LED_BUILTIN"
- board text added: "MISO1"
- board text added: "MISO5"
- board text added: "MOSI1"
- board text added: "MOSI5"
- board text added: "PA10"
- board text added: "PA15"
- board text added: "PC7"
- board text added: "PD13"
- board text added: "PF14"
- board text added: "PF7"
- board text added: "PG13"
- board text added: "PG15"
- board text added: "RX1"
- board text added: "RX2"
- board text added: "RX3"
- board text added: "RX4"
- board text added: "SCL1"
- board text added: "SCL2"
- board text added: "SDA1"
- board text added: "SDA2"
- board text added: "SolarVision Mower STM32N6 Board Rev A - 03/2026 SolarVisionMower.github.io"
- board text added: "TX1"
- board text added: "TX2"
- board text added: "TX3"
- board text added: "TX4"
- board text added: "~{CS}1"
- board text added: "~{CS}5"
