File: Hardware/UWB_CarrierBoard/UWB_CarrierBoard.kicad_sch (KiCad schematic)
At the start: 10 parts, among them J1 Conn_01x09_Socket, J2 Conn_01x09_Socket, U1 DWM1000

Commit message: Finished up the board, generated gerbers, and all other stuffs.
- Added datasheets
- Changed the TVS diode to smth JLC had in stock
- Added pin labels
- Obviously regenerated the gerbers n related stuff
Parts:
- removed D2: D_TVS, Diode_SMD:D_0805_2012Metric, symbol Device:D_TVS
- added D1: D_TVS, Package_TO_SOT_SMD:SOT-723, symbol Device:D_TVS_Dual_AAC
Connections:
- net +5V: now also D1.1 (A1), D1.2 (A2)
- net GND: now also D1.3 (common)
Changed lines of the file:
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@@
+	)
+	(junction
+		(at 26.67 121.92)
+		(diameter 0)
+		(color 0 0 0 0)
 	)
 	(junction
@@
 	)
 	(junction
-		(at 76.2 129.54)
+		(at 36.83 139.7)
 		(diameter 0)
 		(color 0 0 0 0)
 	)
 	(junction
-		(at 36.83 139.7)
+		(at 76.2 129.54)
 		(diameter 0)
 		(color 0 0 0 0)
@@
 	(wire
 		(pts
+			(xy 24.13 121.92) (xy 26.67 121.92)
+		)
+		(stroke
+			(width 0)
+			(type default)
+		)
+	)
+	(wire
+		(pts
 			(xy 123.19 71.12) (xy 130.81 71.12)
 		)
@@
 	(wire
 		(pts
-			(xy 27.94 121.92) (xy 36.83 121.92)
-		)
-		(stroke
-			(width 0)
-			(type default)
-		)
-	)
-	(wire
-		(pts
 			(xy 40.64 129.54) (xy 40.64 121.92)
 		)
@@
 	(wire
 		(pts
+			(xy 24.13 139.7) (xy 26.67 139.7)
+		)
+		(stroke
+			(width 0)
+			(type default)
+		)
+	)
+	(wire
+		(pts
 			(xy 86.36 81.28) (xy 86.36 85.09)
 		)
@@
 	(wire
 		(pts
-			(xy 27.94 139.7) (xy 36.83 139.7)
+			(xy 20.32 143.51) (xy 36.83 143.51)
 		)
 		(stroke
@@
 		)
 	)
-	(wire
-		(pts
-			(xy 27.94 137.16) (xy 27.94 139.7)
-		)
-		(stroke
-			(width 0)
-			(type default)
-		)
-	)
 	(bus
 		(pts
@@
 	(wire
 		(pts
+			(xy 20.32 130.81) (xy 20.32 143.51)
+		)
+		(stroke
+			(width 0)
+			(type default)
+		)
+	)
+	(wire
+		(pts
 			(xy 87.63 127) (xy 87.63 121.92)
 		)
@@
 	(wire
 		(pts
+			(xy 26.67 139.7) (xy 26.67 121.92)
+		)
+		(stroke
+			(width 0)
+			(type default)
+		)
+	)
+	(wire
+		(pts
 			(xy 135.89 58.42) (xy 142.24 58.42)
 		)
@@
 		)
 	)
+	(wire
+		(pts
+			(xy 36.83 143.51) (xy 36.83 139.7)
+		)
+		(stroke
+			(width 0)
+			(type default)
+		)
+	)
+	(wire
+		(pts
+			(xy 26.67 121.92) (xy 36.83 121.92)
+		)
+		(stroke
+			(width 0)
+			(type default)
+		)
+	)
 	(bus
 		(pts
@@
 		(pts
 			(xy 156.21 55.88) (xy 156.21 58.42)
-		)
-		(stroke
-			(width 0)
-			(type default)
-		)
-	)
-	(wire
-		(pts
-			(xy 27.94 129.54) (xy 27.94 121.92)
 		)
 		(stroke
@@
 	)
 	(symbol
-		(lib_id "Device:D_TVS")
-		(at 27.94 133.35 90)
-		(unit 1)
-		(exclude_from_sim no)
-		(in_bom yes)
-		(on_board yes)
-		(dnp no)
-		(fields_autoplaced yes)
-		(property "Reference" "D2"
-			(at 30.48 132.0799 90)
-			(effects
-				(font
-					(size 1.27 1.27)
-				)
-				(justify right)
-			)
-		)
-		(property "Value" "D_TVS"
-			(at 30.48 134.6199 90)
-			(effects
-				(font
-					(size 1.27 1.27)
-				)
-				(justify right)
-			)
-		)
-		(property "Footprint" "Diode_SMD:D_0805_2012Metric"
-			(at 27.94 133.35 0)
-			(effects
-				(font
-					(size 1.27 1.27)
-				)
-				(hide yes)
-			)
-		)
-		(property "Datasheet" "~"
-			(at 27.94 133.35 0)
-			(effects
-				(font
-					(size 1.27 1.27)
-				)
-				(hide yes)
-			)
-		)
-		(property "Description" "Bidirectional transient-voltage-suppression diode"
-			(at 27.94 133.35 0)
-			(effects
-				(font
-					(size 1.27 1.27)
-				)
-				(hide yes)
-			)
-		)
-		(pin "2"
-		)
-		(pin "1"
-		)
-		(instances
-			(project "UWB_CarrierBoard"
-				(path "/91b394b3-3dfa-46b7-845b-422e1bc9b943"
-					(reference "D2")
-					(unit 1)
-				)
-			)
-		)
-	)
-	(symbol
 		(lib_id "symbols:DWM1000")
 		(at 57.15 63.5 0)
@@
 					(unit 1)
 				)
+			)
+		)
+	)
+	(symbol
+		(lib_id "Device:D_TVS_Dual_AAC")
+		(at 24.13 130.81 270)
+		(unit 1)
+		(exclude_from_sim no)
+		(in_bom yes)
+		(on_board yes)
+		(dnp no)
+		(fields_autoplaced yes)
+		(property "Reference" "D1"
+			(at 26.67 129.5399 90)
+			(effects
+				(font
+					(size 1.27 1.27)
+				)
+				(justify left)
+			)
+		)
+		(property "Value" "D_TVS"
+			(at 26.67 132.0799 90)
+			(effects
+				(font
+					(size 1.27 1.27)
+				)
+				(justify left)
+			)
+		)
+		(property "Footprint" "Package_TO_SOT_SMD:SOT-723"
+			(at 24.13 127 0)
+			(effects
+				(font
+					(size 1.27 1.27)
+				)
+				(hide yes)
+			)
+		)
+		(property "Datasheet" "~"
+			(at 24.13 127 0)
+			(effects
+				(font
+					(size 1.27 1.27)
+				)
+				(hide yes)
+			)
+		)
+		(property "Description" "Bidirectional dual transient-voltage-suppression diode, center on pin 3"
+			(at 24.13 130.81 0)
+			(effects
+				(font
+					(size 1.27 1.27)
+				)
+				(hide yes)
+			)
+		)
+		(pin "2"
+		)
+		(pin "1"
+		)
+		(pin "3"
+		)
+		(instances
+			(project ""
+				(path "/91b394b3-3dfa-46b7-845b-422e1bc9b943"
+					(reference "D1")
+					(unit 1)
+				)
